Commit message: fix CoM and mass values

File: lara.xacro (robot description, xacro)
@@ -3,8 +3,4 @@
     <link name="base_link">
     </link>
-    <joint name="base_link_to_chassis" type="fixed">
-        <parent link="base_link"/>
-        <child link="chassis"/>
-    </joint>
     <link name="chassis">
         <visual>
@@ -19,8 +15,13 @@
         </collision>
         <inertial>
-            <mass value="100"/>
+            <mass value="20"/>
             <inertia ixx="0.4" ixy="0.0" ixz="0.0" iyy="0.4" iyz="0.0" izz="0.2"/>
+            <origin xyz="0 -0.15 0" rpy="0 0 0"/>
         </inertial>
     </link>
+    <joint name="base_link_to_chassis" type="fixed">
+        <parent link="base_link"/>
+        <child link="chassis"/>
+    </joint>
     <link name="link_1">
         <visual>
@@ -35,5 +36,5 @@
         </collision>
         <inertial>
-            <mass value="10"/>
+            <mass value="0.1"/>
             <inertia ixx="0.4" ixy="0.0" ixz="0.0" iyy="0.4" iyz="0.0" izz="0.2"/>
         </inertial>
@@ -58,5 +59,5 @@
         </collision>
         <inertial>
-            <mass value="10"/>
+            <mass value="0.1"/>
             <inertia ixx="0.4" ixy="0.0" ixz="0.0" iyy="0.4" iyz="0.0" izz="0.2"/>
         </inertial>
@@ -81,5 +82,5 @@
         </collision>
         <inertial>
-            <mass value="10"/>
+            <mass value="0.1"/>
             <inertia ixx="0.4" ixy="0.0" ixz="0.0" iyy="0.4" iyz="0.0" izz="0.2"/>
         </inertial>
@@ -104,5 +105,5 @@
         </collision>
         <inertial>
-            <mass value="10"/>
+            <mass value="0.1"/>
             <inertia ixx="0.4" ixy="0.0" ixz="0.0" iyy="0.4" iyz="0.0" izz="0.2"/>
         </inertial>
@@ -127,5 +128,5 @@
         </collision>
         <inertial>
-            <mass value="10"/>
+            <mass value="0.1"/>
             <inertia ixx="0.4" ixy="0.0" ixz="0.0" iyy="0.4" iyz="0.0" izz="0.2"/>
         </inertial>
@@ -150,5 +151,5 @@
         </collision>
         <inertial>
-            <mass value="10"/>
+            <mass value="0.05"/>
             <inertia ixx="0.4" ixy="0.0" ixz="0.0" iyy="0.4" iyz="0.0" izz="0.2"/>
         </inertial>
@@ -173,5 +174,5 @@
         </collision>
         <inertial>
-            <mass value="10"/>
+            <mass value="0.05"/>
             <inertia ixx="0.4" ixy="0.0" ixz="0.0" iyy="0.4" iyz="0.0" izz="0.2"/>
         </inertial>
