Commit message: Adding wheels. Moves but still needs true inertial vals

File: urdf/lara.xacro (robot description, xacro)
@@ -1,4 +1,7 @@
 <?xml version="1.0"?>
 <robot xmlns:xacro="http://www.ros.org/wiki/xacro" name="lara">
+    <xacro:include filename="$(find lara_model)/urdf/simulation/gazebo_base.xacro" />
+    <xacro:include filename="$(find lara_model)/urdf/simulation/gazebo_laser.xacro" />
+    <xacro:include filename="$(find lara_model)/urdf/pioneer3dx_wheel.xacro" />
     <link name="base_link">
     </link>
@@ -8,4 +11,5 @@
                 <mesh filename="package://lara_model/objs/Chassis.obj"/>
             </geometry>
+            <origin xyz="0 0 0" rpy="0 0 ${-3.14159265/2}"/>
         </visual>
         <collision>
@@ -13,9 +17,10 @@
                 <mesh filename="package://lara_model/objs/Chassis.obj"/>
             </geometry>
+            <origin xyz="0 0 0" rpy="0 0 ${-3.14159265/2}"/>
         </collision>
         <inertial>
             <mass value="20"/>
             <inertia ixx="0.4" ixy="0.0" ixz="0.0" iyy="0.4" iyz="0.0" izz="0.2"/>
-            <origin xyz="0 -0.15 0" rpy="0 0 0"/>
+            <origin xyz="-0.15 0 0" rpy="0 0 ${-3.14159265/2}"/>
         </inertial>
     </link>
@@ -24,4 +29,8 @@
         <child link="chassis"/>
     </joint>
+    <!-- WHEELS -->
+    <xacro:p3dx_wheel suffix="left" parent="chassis" reflect="1"/>
+    <xacro:p3dx_wheel suffix="right" parent="chassis" reflect="-1"/>
+    <!-- MANIPULATOR -->
     <link name="link_1">
         <visual>
@@ -185,3 +194,34 @@
         <origin rpy="0 0 0" xyz="-0.03715033 0.05965715 0.0045"/>
     </joint>
+  <!-- SENSORS -->
+  <joint name="hokuyo_joint" type="fixed">
+    <axis xyz="0 1 0" />
+    <origin xyz="0 0.075 -0.05" rpy="0 0 0"/>
+    <parent link="chassis"/>
+    <child link="hokuyo_link"/>
+  </joint>
+  <!-- Hokuyo Laser -->
+  <link name="hokuyo_link">
+    <collision>
+      <origin xyz="0 0 0" rpy="0 0 0"/>
+      <geometry>
+    <box size="0.05 0.05 0.07"/>
+      </geometry>
+    </collision>
+    <!-- TODO: USE HOKUYO MODEL  -->
+    <!-- <visual name="visual">
+    <origin xyz="0 0.075 -0.05" rpy="0 0 0"/>
+    <geometry>
+        <box size="0.05 0.05 0.07" />
+    </geometry>
+    </visual> -->
+    <inertial>
+      <mass value="1e-5" />
+      <origin xyz="0 0 0" rpy="0 0 0"/>
+      <inertia ixx="1e-6" ixy="0" ixz="0" iyy="1e-6" iyz="0" izz="1e-6" />
+    </inertial>
+  </link>
+  <!-- Plugins -->
+  <xacro:gazebo_base reference="p3dx"/>
+  <xacro:gazebo_laser reference="hokuyo_link"/>
 </robot>

Commit message: tuning CoM and adding center whell

File: urdf/lara.xacro (robot description, xacro)
@@ -22,5 +22,5 @@
             <mass value="20"/>
             <inertia ixx="0.4" ixy="0.0" ixz="0.0" iyy="0.4" iyz="0.0" izz="0.2"/>
-            <origin xyz="-0.15 0 0" rpy="0 0 ${-3.14159265/2}"/>
+            <origin xyz="-0.20 0 0" rpy="0 0 ${-3.14159265/2}"/>
         </inertial>
     </link>
@@ -30,167 +30,95 @@
     </joint>
     <!-- WHEELS -->
-    <xacro:p3dx_wheel suffix="left" parent="chassis" reflect="1"/>
-    <xacro:p3dx_wheel suffix="right" parent="chassis" reflect="-1"/>
-    <!-- MANIPULATOR -->
-    <link name="link_1">
+    <xacro:p3dx_wheel suffix="right" parent="chassis" reflect="1"/>
+    <xacro:p3dx_wheel suffix="left" parent="chassis" reflect="-1"/>
+    <!-- Swivel -->
+    <link name="swivel">
+        <inertial>
+        <mass value="0.1"/>
+        <origin xyz="0 0 0"/>
+        <inertia ixx="0.01" ixy="0" ixz="0"
+                iyy="0.01" iyz="0" izz="0.01"/>
+        </inertial>
         <visual>
-            <geometry>
-                <mesh filename="package://lara_model/objs/Link1.obj"/>
-            </geometry>
+        <origin xyz="0 0 0" rpy="0 0 0"/>
+        <geometry name="pioneer_geom">
+            <mesh filename="package://lara_model/meshes/swivel.stl"/>
+        </geometry>
+        <material name="swivel">
+            <color rgba="0.5 0.5 0.5 1"/>
+        </material>
+        </visual>
+    </link>
+    <gazebo reference="swivel">
+        <material value="Gazebo/Black"/>
+    </gazebo>
+    <joint name="base_swivel_joint" type="continuous">
+        <origin xyz="-0.27 0 -0.19" rpy="0 0 0"/>
+        <axis xyz="0 0 1"/>
+        <limit effort="100" velocity="100" k_velocity="0" />
+        <joint_properties damping="0.0" friction="0.0" />
+        <parent link="chassis"/>
+        <child link="swivel"/>
+    </joint>
+    <!-- Center Wheel + Hubcap -->
+    <link name="center_hubcap">
+        <inertial>
+        <mass value="0.01"/>
+        <origin xyz="0 0 0"/>
+        <inertia ixx="0.012411765597" ixy="-0.000711733678" ixz="0.00050272983"
+                iyy="0.015218160428" iyz="-0.000004273467" izz="0.011763977943"/>
+        </inertial>
+        <visual>
+        <origin xyz="0 0 0" rpy="0 0 0"/>
+        <geometry name="pioneer_geom">
+            <mesh filename="package://lara_model/meshes/center_hubcap.stl"/>
+        </geometry>
+        <material name="swivel">
+            <color rgba="0.5 0.5 0.5 1"/>
+        </material>
+        </visual>
+    </link>
+    <gazebo reference="center_hubcap">
+        <material value="Gazebo/Black"/>
+    </gazebo>
+    <joint name="swivel_hubcap_joint" type="continuous">
+        <origin xyz="-0.026 0 -0.016" rpy="0 0 0"/>
+        <axis xyz="0 1 0"/>
+        <anchor xyz="0 0 0"/>
+        <limit effort="100" velocity="100" k_velocity="0" />
+        <joint_properties damping="0.0" friction="0.0" />
+        <parent link="swivel"/>
+        <child link="center_wheel"/>
+    </joint>
+    <link name="center_wheel">
+        <inertial>
+        <mass value="0.1"/>
+        <origin xyz="0 0 0"/>
+        <inertia ixx="0.012411765597" ixy="-0.000711733678" ixz="0.00050272983"
+                iyy="0.015218160428" iyz="-0.000004273467" izz="0.011763977943"/>
+        </inertial>
+        <visual>
+        <origin xyz="0 0 0" rpy="0 0 0"/>
+        <geometry name="pioneer_geom">
+            <mesh filename="package://lara_model/meshes/center_wheel.stl"/>
+        </geometry>
+        <material name="WheelBlack">
+            <color rgba="0.117 0.117 0.117 1"/>
+        </material>
         </visual>
         <collision>
-            <geometry>
-                <mesh filename="package://lara_model/objs/Link1.obj"/>
-            </geometry>
+        <origin xyz="0 0 0" rpy="${-3.1415927/2.0} 0 0"/>
+        <geometry>
+            <cylinder radius="0.0375" length="0.0314"/>
+        </geometry>
         </collision>
-        <inertial>
-            <mass value="0.1"/>
-            <inertia ixx="0.4" ixy="0.0" ixz="0.0" iyy="0.4" iyz="0.0" izz="0.2"/>
-        </inertial>
     </link>
-    <joint name="chassis_to_link_1" type="revolute">
-        <axis xyz="0 0 1"/>
-        <limit effort="1000.0" lower="${-pi/2}" upper="${pi/2}" velocity="0.5"/>
-        <parent link="chassis"/>
-        <child link="link_1"/>
-        <origin rpy="0 0 0" xyz="-0.0000005953 -0.05506373 0.36944"/>
-    </joint>
-    <link name="link_2">
-        <visual>
-            <geometry>
-                <mesh filename="package://lara_model/objs/Link2.obj"/>
-            </geometry>
-        </visual>
-        <collision>
-            <geometry>
-                <mesh filename="package://lara_model/objs/Link2.obj"/>
-            </geometry>
-        </collision>
-        <inertial>
-            <mass value="0.1"/>
-            <inertia ixx="0.4" ixy="0.0" ixz="0.0" iyy="0.4" iyz="0.0" izz="0.2"/>
-        </inertial>
-    </link>
-    <joint name="link_1_to_link_2" type="revolute">
-        <axis xyz="1 0 0"/>
-        <limit effort="1000.0" lower="${-pi/2}" upper="${pi/2}" velocity="0.5"/>
-        <parent link="link_1"/>
-        <child link="link_2"/>
-        <origin rpy="0 0 0" xyz="0 0.145 0"/>
-    </joint>
-    <link name="link_3">
-        <visual>
-            <geometry>
-                <mesh filename="package://lara_model/objs/Link3.obj"/>
-            </geometry>
-        </visual>
-        <collision>
-            <geometry>
-                <mesh filename="package://lara_model/objs/Link3.obj"/>
-            </geometry>
-        </collision>
-        <inertial>
-            <mass value="0.1"/>
-            <inertia ixx="0.4" ixy="0.0" ixz="0.0" iyy="0.4" iyz="0.0" izz="0.2"/>
-        </inertial>
-    </link>
-    <joint name="link_2_to_link_3" type="revolute">
-        <axis xyz="1 0 0"/>
-        <limit effort="1000.0" lower="${-pi/2}" upper="${pi/2}" velocity="0.5"/>
-        <parent link="link_2"/>
-        <child link="link_3"/>
-        <origin rpy="0 0 0" xyz="0.0068396853 0.27 0"/>
-    </joint>
-    <link name="link_4">
-        <visual>
-            <geometry>
-                <mesh filename="package://lara_model/objs/Link4.obj"/>
-            </geometry>
-        </visual>
-        <collision>
-            <geometry>
-                <mesh filename="package://lara_model/objs/Link4.obj"/>
-            </geometry>
-        </collision>
-        <inertial>
-            <mass value="0.1"/>
-            <inertia ixx="0.4" ixy="0.0" ixz="0.0" iyy="0.4" iyz="0.0" izz="0.2"/>
-        </inertial>
-    </link>
-    <joint name="link_3_to_link_4" type="revolute">
-        <axis xyz="0 1 0"/>
-        <limit effort="1000.0" lower="${-pi/2}" upper="${pi/2}" velocity="0.5"/>
-        <parent link="link_3"/>
-        <child link="link_4"/>
-        <origin rpy="0 0 0" xyz="0 0 0"/>
-    </joint>
-    <link name="link_5">
-        <visual>
-            <geometry>
-                <mesh filename="package://lara_model/objs/Link5.obj"/>
-            </geometry>
-        </visual>
-        <collision>
-            <geometry>
-                <mesh filename="package://lara_model/objs/Link5.obj"/>
-            </geometry>
-        </collision>
-        <inertial>
-            <mass value="0.1"/>
-            <inertia ixx="0.4" ixy="0.0" ixz="0.0" iyy="0.4" iyz="0.0" izz="0.2"/>
-        </inertial>
-    </link>
-    <joint name="link_4_to_link_5" type="revolute">
-        <axis xyz="1 0 0"/>
-        <limit effort="1000.0" lower="${-pi/2}" upper="${pi/2}" velocity="0.5"/>
-        <parent link="link_4"/>
-        <child link="link_5"/>
-        <origin rpy="0 0 0" xyz="0 0 0"/>
-    </joint>
-    <link name="finger_r">
-        <visual>
-            <geometry>
-                <mesh filename="package://lara_model/objs/FingerR.obj"/>
-            </geometry>
-        </visual>
-        <collision>
-            <geometry>
-                <mesh filename="package://lara_model/objs/FingerR.obj"/>
-            </geometry>
-        </collision>
-        <inertial>
-            <mass value="0.05"/>
-            <inertia ixx="0.4" ixy="0.0" ixz="0.0" iyy="0.4" iyz="0.0" izz="0.2"/>
-        </inertial>
-    </link>
-    <joint name="link_5_to_finger_r" type="revolute">
-        <axis xyz="0 0 1"/>
-        <limit effort="1000.0" lower="${-pi/2}" upper="${pi/2}" velocity="0.5"/>
-        <parent link="link_5"/>
-        <child link="finger_r"/>
-        <origin rpy="0 0 0" xyz="0.03284967 0.05965715 0.0045"/>
-    </joint>
-    <link name="finger_l">
-        <visual>
-            <geometry>
-                <mesh filename="package://lara_model/objs/FingerL.obj"/>
-            </geometry>
-        </visual>
-        <collision>
-            <geometry>
-                <mesh filename="package://lara_model/objs/FingerL.obj"/>
-            </geometry>
-        </collision>
-        <inertial>
-            <mass value="0.05"/>
-            <inertia ixx="0.4" ixy="0.0" ixz="0.0" iyy="0.4" iyz="0.0" izz="0.2"/>
-        </inertial>
-    </link>
-    <joint name="link_5_to_finger_l" type="revolute">
-        <axis xyz="0 0 1"/>
-        <limit effort="1000.0" lower="${-pi/2}" upper="${pi/2}" velocity="0.5"/>
-        <parent link="link_5"/>
-        <child link="finger_l"/>
-        <origin rpy="0 0 0" xyz="-0.03715033 0.05965715 0.0045"/>
+    <gazebo reference="center_wheel">
+        <material value="Gazebo/Black"/>
+    </gazebo>
+    <joint name="center_wheel_joint" type="fixed">
+        <origin xyz="-0.0035 0 -0.001" rpy="0 0 0"/>
+        <parent link="center_wheel"/>
+        <child link="center_hubcap"/>
     </joint>
   <!-- SENSORS -->
